File: ESP-Mini-Base.kicad_pcb (KiCad board)
At the start: 2 copper layers, 76.2 x 47.6 mm, 75 parts, among them IC1 LM2940IMP-5.0_NOPB, J1 Screw_Terminal_01x03, J10 Conn_01x03, J11 Conn_01x16, J12 Conn_01x06, J13 Conn_01x06, J7 Conn_01x02, J8 Conn_01x16, J9 Screw_Terminal_01x03, Q1 AO4402G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

Commit message: minor improvements; updated to KiCAD 8
Routing:
- net GND: track 5.08 -> 0.00 mm, vias 2 -> 30
- net +12V: track 32.3 -> 33.1 mm
- added copper zone on B.Cu, net GND
Other:
- board text added: "ESP-Mini-Base v1.1 (c)github.com/juepi"
- board text removed: "ESP-Mini-Base v1.0 (c)github.com/juepi"
