File: ESP-Mini-Base.kicad_sch (KiCad schematic)
At the start: 75 parts, among them IC1 LM2940IMP-5.0_NOPB, J1 Screw_Terminal_01x03, J10 Conn_01x03, J11 Conn_01x16, J12 Conn_01x06, J13 Conn_01x06, J7 Conn_01x02, J8 Conn_01x16, J9 Screw_Terminal_01x03, Q1 AO4402G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

Commit message: update readme, pictures, schematic usage notes and pdf
Other:
- note added: "3x N-Channel MOSFET Switches max. 5A / 20Vds"
- note added: "5V Linear LDO Voltage Regulator Supports 6.25~26VDC input voltage"
- note added: "ADC Attenuator 5V -> 1.15V, Factor: 0.23"
- note added: "ATTN: Do NOT connect USB power (VBUS) while supplying the ESP through LDO!"
- note added: "ATTN: JP12 and JP13 must be OPENED!"
- note added: "ATTN: always use GND wire on J9 when switching high loads!"
- note added: "Disabled by default short JP14+JP16 / JP15+JP17 to enable"
- note added: "Gates unconnected by default, with ability to re-route them as required short solder jumpers JP6-JP8 as required to use default GPIOs."
- note added: "Level Shifting 3V3 -> 5V"
- note added: "Optional 5V I2C Pullups for D1 Mini"
- note added: "Optional 5V I2C Pullups for S2 Mini"
- note added: "Power Supply Switch 3V3 or 5V max. 2A, disabled by default"
- note added: "Pushbutton"
- note added: "Select voltage to measure through JP5 leave JP5 openend to supply external voltage via J5"
- note added: "Short JP11 to use IO14 as switching signal (active high)"
- note added: "Short JP3 to enable button on IO16"
- note added: "Short JP9 to use IO13 as switching signal (active high)"
- note added: "To enable pullups, short pads 1-3 on JP18."
- note added: "To enable pullups, short pads 1-3 on JP19."
- note added: "To enable pullups, short pads 1-3 on the corresponding jumper pads."
- note added: "Use JP10 to select voltage to be switched by U2"
- note added: "Use if 5V are required when running from single LFP cell (connected directly to 3V3)"
- note added: "short JP13 to enable output voltage short JP12 to supply 5V to ESP."
- note removed: "3x N-Channel MOSFET Switches max. 5A / 20V"
- note removed: "5V Input Linear Voltage Regulator use when powered from 12VDC"
- note removed: "ADC Attenuator 5V -> 1.15V Factor: 0.23"
- note removed: "Gates unconnected by default, with ability to re-route them as required"
- note removed: "Level Shifting 3V3 -> 5V Disabled by default"
- note removed: "Optional I2C Pullups 5V for S2 Mini"
- note removed: "Optional I2C Pullups for D1 Mini"
- note removed: "Optional Pushbutton"
- note removed: "Power Supply Switch 3V3 or 5V Disabled by default"
- note removed: "Use if 5V are required when running from single LFP cell (connected directly to 3V3) JP12 and JP13 must be OPENED!"
Changed lines of the file:
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@@
   (title_block
     (title "Base PCB for ESP* in WEMOS Mini Format")
-    (date "2023-12-17")
+    (date "2023-12-22")
     (rev "1.0")
   )
@@
     (stroke (width 0) (type default))
   )
+  (text "To enable pullups, short pads 1-3 on the corresponding jumper pads."
+    (at 26.67 172.72 0)
+    (effects (font (size 1.27 1.27)) (justify left bottom))
+  )
   (text "SDA for S2 Mini" (at 381 121.92 0)
     (effects (font (size 1.27 1.27)) (justify left bottom))
   )
+  (text "Select voltage to measure through JP5\nleave JP5 openend to supply\nexternal voltage via J5"
+    (at 62.23 233.68 0)
+    (effects (font (size 1.27 1.27)) (justify left bottom))
+  )
   (text "MCU Socket\nCompartible with\nWEMOS S2 Mini\nWEMOS D1 Mini"
     (at 177.8 45.72 0)
@@
     (effects (font (size 1.27 1.27)) (justify left bottom))
   )
-  (text "Optional I2C Pullups\nfor D1 Mini" (at 355.6 157.48 0)
+  (text "Optional 5V I2C Pullups for D1 Mini" (at 355.6 154.94 0)
     (effects (font (size 1.27 1.27) italic) (justify left bottom))
   )
@@
     (effects (font (size 1.27 1.27) italic) (justify left bottom))
   )
-  (text "5V Input Linear Voltage Regulator\nuse when powered from 12VDC"
-    (at 208.28 229.87 0)
+  (text "5V Linear LDO Voltage Regulator\nSupports 6.25~26VDC input voltage"
+    (at 208.28 226.06 0)
     (effects (font (size 2 2) italic) (justify left bottom))
   )
-  (text "Level Shifting 3V3 -> 5V\nDisabled by default" (at 306.07 50.8 0)
+  (text "Level Shifting 3V3 -> 5V" (at 306.07 50.8 0)
     (effects (font (size 2 2) italic) (justify left bottom))
   )
+  (text "Disabled by default\nshort JP14+JP16 / JP15+JP17 to enable"
+    (at 306.07 55.88 0)
+    (effects (font (size 1.27 1.27)) (justify left bottom))
+  )
   (text "SS/IO15" (at 153.67 90.17 0)
     (effects (font (size 1.27 1.27)) (justify left bottom))
@@
     (effects (font (size 1.27 1.27)) (justify left bottom))
   )
+  (text "Short JP9 to use IO13 as switching signal (active high)"
+    (at 113.03 229.87 0)
+    (effects (font (size 1.27 1.27)) (justify left bottom))
+  )
   (text "IO7" (at 375.92 119.38 0)
     (effects (font (size 1.27 1.27)) (justify left bottom))
@@
     (effects (font (size 1.27 1.27)) (justify left bottom))
   )
-  (text "Power Supply Switch 3V3 or 5V\nDisabled by default" (at 116.84 148.59 0)
+  (text "Power Supply Switch 3V3 or 5V\nmax. 2A, disabled by default"
+    (at 116.84 148.59 0)
     (effects (font (size 2 2) italic) (justify left bottom))
   )
@@
     (effects (font (size 1.27 1.27)) (justify left bottom))
   )
+  (text "Short JP11 to use IO14 as switching signal (active high)"
+    (at 116.84 153.67 0)
+    (effects (font (size 1.27 1.27)) (justify left bottom))
+  )
   (text "for D1 Mini" (at 66.04 180.34 0)
     (effects (font (size 1.27 1.27) italic) (justify left bottom))
@@
     (effects (font (size 1.27 1.27)) (justify left bottom))
   )
-  (text "Gates unconnected by default, with ability to re-route them as required"
-    (at 36.83 31.75 0)
+  (text "Gates unconnected by default, with ability to re-route them as required\nshort solder jumpers JP6-JP8 as required to use default GPIOs."
+    (at 36.83 33.02 0)
+    (effects (font (size 1.27 1.27)) (justify left bottom))
+  )
+  (text "Short JP3 to enable button on IO16" (at 31.75 130.81 0)
     (effects (font (size 1.27 1.27)) (justify left bottom))
   )
@@
     (effects (font (size 1.27 1.27)) (justify left bottom))
   )
+  (text "ATTN: Do NOT connect USB power (VBUS) while supplying the ESP through LDO!"
+    (at 208.28 233.68 0)
+    (effects (font (size 1.27 1.27) (thickness 0.254) bold italic) (justify left bottom))
+  )
   (text "IO4/SDA" (at 222.25 77.47 0)
     (effects (font (size 1.27 1.27)) (justify left bottom))
   )
-  (text "Solid-State Relays AC/DC\nmax. 500mA / 48Vpp" (at 113.03 229.87 0)
+  (text "To enable pullups, short pads 1-3 on JP18." (at 355.6 80.01 0)
+    (effects (font (size 1.27 1.27)) (justify left bottom))
+  )
+  (text "Use JP10 to select voltage to be switched by U2" (at 116.84 151.13 0)
+    (effects (font (size 1.27 1.27)) (justify left bottom))
+  )
+  (text "To enable pullups, short pads 1-3 on JP19." (at 355.6 157.48 0)
+    (effects (font (size 1.27 1.27)) (justify left bottom))
+  )
+  (text "Solid-State Relays AC/DC\nmax. 500mA / 48Vpp" (at 113.03 227.33 0)
     (effects (font (size 2 2) italic) (justify left bottom))
   )
-  (text "Optional I2C Pullups 5V\nfor S2 Mini" (at 355.6 80.01 0)
+  (text "Optional 5V I2C Pullups for S2 Mini" (at 355.6 77.47 0)
     (effects (font (size 1.27 1.27) italic) (justify left bottom))
   )
@@
     (effects (font (size 1.27 1.27)) (justify left bottom))
   )
-  (text "3x N-Channel MOSFET Switches\nmax. 5A / 20V" (at 36.83 27.94 0)
+  (text "3x N-Channel MOSFET Switches\nmax. 5A / 20Vds" (at 36.83 27.94 0)
     (effects (font (size 2 2) italic) (justify left bottom))
   )
-  (text "Use if 5V are required when running from single LFP cell\n(connected directly to 3V3)\nJP12 and JP13 must be OPENED!"
-    (at 190.5 162.56 0)
+  (text "Use if 5V are required when running from single LFP cell\n(connected directly to 3V3)"
+    (at 186.69 160.02 0)
     (effects (font (size 1.27 1.27)) (justify left bottom))
   )
@@
     (effects (font (size 1.27 1.27)) (justify left bottom))
   )
+  (text "short JP13 to enable output voltage\nshort JP12 to supply 5V to ESP."
+    (at 208.28 231.14 0)
+    (effects (font (size 1.27 1.27)) (justify left bottom))
+  )
   (text "5V" (at 222.25 97.79 0)
     (effects (font (size 1.27 1.27)) (justify left bottom))
@@
     (effects (font (size 1.27 1.27)) (justify left bottom))
   )
-  (text "Optional Pushbutton" (at 31.75 129.54 0)
+  (text "Pushbutton" (at 31.75 128.27 0)
     (effects (font (size 2 2) italic) (justify left bottom))
   )
@@
     (effects (font (size 1.27 1.27)) (justify left bottom))
   )
-  (text "Optional Header for Boost Converter 3V3 -> 5V" (at 179.07 153.67 0)
+  (text "Optional Header for Boost Converter 3V3 -> 5V" (at 186.69 154.94 0)
     (effects (font (size 2 2) italic) (justify left bottom))
   )
@@
     (effects (font (size 1.27 1.27)) (justify left bottom))
   )
-  (text "Optional I2C Pullups 3V3" (at 33.02 171.45 0)
+  (text "ATTN: always use GND wire on J9 when switching high loads!"
+    (at 36.83 35.56 0)
+    (effects (font (size 1.27 1.27) bold italic) (justify left bottom))
+  )
+  (text "Optional I2C Pullups 3V3" (at 26.67 170.18 0)
     (effects (font (size 2 2) italic) (justify left bottom))
   )
-  (text "ADC Attenuator\n5V -> 1.15V\nFactor: 0.23" (at 71.12 232.41 0)
+  (text "ATTN: JP12 and JP13 must be OPENED!" (at 186.69 162.56 0)
+    (effects (font (size 1.27 1.27) (thickness 0.254) bold italic) (justify left bottom))
+  )
+  (text "ADC Attenuator\n5V -> 1.15V, Factor: 0.23" (at 62.23 227.33 0)
     (effects (font (size 2 2) italic) (justify left bottom))
   )
@@
   )
   (symbol (lib_id "power:+3.3V") (at 119.38 158.75 0) (unit 1)
-    (in_bom yes) (on_board yes) (dnp no) (fields_autoplaced)
+    (in_bom yes) (on_board yes) (dnp no)
     (property "Reference" "#PWR0119" (at 119.38 162.56 0)
       (effects (font (size 1.27 1.27)) hide)
     )
-    (property "Value" "+3.3V" (at 119.38 153.67 0)
+    (property "Value" "+3.3V" (at 119.38 154.94 0)
       (effects (font (size 1.27 1.27)))
     )

Commit message: fixed typo
Other:
- note added: "MCU Socket Compatible with WEMOS S2 Mini WEMOS D1 Mini"
- note removed: "MCU Socket Compartible with WEMOS S2 Mini WEMOS D1 Mini"
Changed lines of the file:
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@@
     (effects (font (size 1.27 1.27)) (justify left bottom))
   )
-  (text "MCU Socket\nCompartible with\nWEMOS S2 Mini\nWEMOS D1 Mini"
+  (text "MCU Socket\nCompatible with\nWEMOS S2 Mini\nWEMOS D1 Mini"
     (at 177.8 45.72 0)
     (effects (font (size 2 2) italic) (justify left bottom))

Commit message: minor improvements; updated to KiCAD 8
Parts:
- H1, H2, J1, J10, J11, J12, J13, J14, J2, J3, J4, J5, J6, J7, J8, J9, JP1, JP10, JP18, JP19, JP2, JP4, JP5, U3: now left out of the parts list
